Commit message: upload new branch - ROS world complete

File: install/robot/share/robot/urdf/robot.urdf (robot description, URDF)
Before this commit: robot robot, 6 links, 5 joints
Links:
- link base: geometry collision mesh filename=package://robot/meshes/base_link_PR.stl; visual mesh filename=package://robot/meshes/base_link.stl
